File: projet/projet/projet.kicad_pcb (KiCad board)
At the start: 2 copper layers, 98.5 x 93 mm, 18 parts, among them SW1 SW_Push, U1 LilyGo-T-A7670E-R2, U2 MPU6050-Breakout

Commit message: Finalisation des fichiers gerbers
Finalisation des fichiers gerbers
Parts:
- moved U2 49.5 mm to (144.0, 85.5)
- moved U1 7.09 mm to (109.2, 89.8)
- moved RV1 6.50 mm to (132.0, 53.5), turned to -90 degrees
- moved RV2 4.63 mm to (103.5, 55.0), turned to 0 degrees
Routing:
- net +3.3V: track 0.00 -> 75.7 mm
- net Net-(U1-IO35/ADC7): track 0.00 -> 46.3 mm
- net Net-(U1-IO27/TOUCH7): track 0.00 -> 36.3 mm
- net Net-(U1-SCL/IO22): track 0.00 -> 28.4 mm
- net Net-(U1-IO34/ADC6): track 0.00 -> 27.1 mm
- net Net-(U1-SDA/IO21): track 0.00 -> 24.8 mm
- net Net-(U1-IO12/TOUCH5): track 0.00 -> 19.3 mm
- net Net-(U1-IO15/TOUCH3): track 0.00 -> 18.3 mm
- net Net-(U1-IO13/TOUCH4): track 0.00 -> 14.9 mm
- net Net-(U1-IO14/TOUCH6): track 0.00 -> 13.8 mm
- net Net-(D3-A): track 0.00 -> 5.69 mm
- net Net-(D2-A): track 0.00 -> 5.19 mm
- net Net-(D1-A): track 0.00 -> 5.00 mm
- net Net-(D4-A): track 0.00 -> 4.69 mm
- added copper zone on B.Cu, net GND
- added copper zone on F.Cu, net GND
